File: project/project.kicad_pcb (KiCad board)
At the start: 2 copper layers, 80 x 165 mm, 19 parts, among them J1 Conn_01x02_Pin, J2 Conn_02x07_Odd_Even, J5 12V

Commit message: added latch
Parts:
- removed REF**: module_ina219, usini_sensors:module_ina219
- added J3: Conn_01x02, Connector_PinHeader_2.54mm:PinHeader_1x02_P2.54mm_Vertical, F.Cu at (202.7, 119.0)
- added Q1: IRF4905, Package_TO_SOT_THT:TO-220-3_Vertical, F.Cu at (193.3, 75.0)
- added Q2: NPN, Package_TO_SOT_THT:TO-92_HandSolder, F.Cu at (184.9, 78.9)
- added R1: 10k, Resistor_THT:R_Axial_DIN0309_L9.0mm_D3.2mm_P12.70mm_Horizontal, F.Cu at (181.8, 111.2)
- added R2: 10k, Resistor_THT:R_Axial_DIN0309_L9.0mm_D3.2mm_P12.70mm_Horizontal, F.Cu at (181.8, 116.0)
- added R3: 4.7k, Resistor_THT:R_Axial_DIN0309_L9.0mm_D3.2mm_P12.70mm_Horizontal, F.Cu at (181.8, 120.7)
- added SW1: SW_Push, Button_Switch_THT:SW_PUSH-12mm, F.Cu at (207.5, 51.0)
- added U1: module_ina219, usini_sensors:module_ina219, F.Cu at (183.9, 102.6)
- J1: value Conn_01x02_Pin -> Conn_01x03; footprint Connector_PinHeader_2.54mm:PinHeader_1x02_P2.54mm_Vertical -> Connector_PinHeader_2.54mm:PinHeader_1x03_P2.54mm_Vertical
- moved J2 158.0 mm to (185.2, 57.8)
- moved Motor2 133.1 mm to (174.2, 93.5), turned to 0 degrees
- moved Motor1 132.7 mm to (174.2, 85.7), turned to 0 degrees
- moved StepDown_5V1 83.6 mm to (148.4, 71.0)
- moved Motor4 77.8 mm to (174.2, 109.1), turned to 0 degrees
- moved Motor3 77.5 mm to (174.2, 101.3), turned to 0 degrees
- moved J1 67.2 mm to (203.9, 73.3)
- moved C5 46.3 mm to (203.2, 112.8)
- moved C1 35.2 mm to (198.2, 110.1)
- moved C2 35.2 mm to (198.2, 112.6)
- moved C3 35.2 mm to (198.2, 115.1)
- moved C4 35.2 mm to (198.2, 117.7)
- moved C6 35.2 mm to (198.2, 120.2)
- moved C7 35.2 mm to (198.2, 122.7)
- moved J5 31.2 mm to (175.1, 116.5)
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Connections:
- J1 pad 1: GND -> /PowLatch
- J5 pad +: (no net) -> Net-(J5-Pin_1)
- J5 pad -: (no net) -> GND
Other:
- outline, holes or cut-outs redrawn

Commit message: last-update
Parts:
- added 1A: 1A, byRadu:OPM_Kuoyuh_91, F.Cu at (34.0, 129.1)
- added 1A: 1A, byRadu:OPM_Kuoyuh_91, F.Cu at (100.0, 129.1)
- moved SW1 213.2 mm to (42.5, 186.0), turned to 90 degrees
- moved C3 154.0 mm to (46.0, 91.5)
- moved Q2 151.9 mm to (71.0, 179.5)
- moved J1 150.7 mm to (57.5, 37.5), turned to 180 degrees
- moved C4 149.5 mm to (51.0, 91.5), turned to 180 degrees
- moved J3 145.6 mm to (84.5, 34.0)
- moved Q1 145.0 mm to (80.0, 165.5)
- moved C6 141.4 mm to (61.0, 86.0), turned to 90 degrees
- moved C5 134.7 mm to (85.0, 177.5), turned to -90 degrees
- moved R3 129.9 mm to (63.0, 173.3), turned to -90 degrees
- moved R1 129.3 mm to (75.8, 185.5)
- moved Motor4 128.7 mm to (45.5, 112.0), turned to -90 degrees
- moved Motor3 128.7 mm to (45.5, 102.5), turned to -90 degrees
- moved C7 122.1 mm to (81.2, 87.8), turned to 90 degrees
- moved U1 119.5 mm to (75.7, 153.5)
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Connections:
- Driver1 pad 1: /VM -> Net-(Driver1-VM)
- Driver2 pad 1: /VM -> Net-(Driver2-VM)
Routing:
- net Net-(U1-VIN-): track 0.00 -> 180.1 mm, vias 0 -> 4
- net /PowLatch: track 0.00 -> 168.3 mm, vias 0 -> 2
- net /VM: track 0.00 -> 159.0 mm, vias 0 -> 6
- net Net-(J3-Pin_1): track 0.00 -> 147.2 mm
- net Net-(J3-Pin_2): track 0.00 -> 145.8 mm, vias 0 -> 4
- net /VCC: track 0.00 -> 145.0 mm
- net Net-(Driver2-VM): track 0.00 -> 84.4 mm, vias 0 -> 4
- net Net-(Driver1-VM): track 0.00 -> 71.4 mm, vias 0 -> 2
- net Net-(Q1-G): track 0.00 -> 66.1 mm
- net /STANDBY: track 0.00 -> 56.8 mm, vias 0 -> 4
- net Net-(J1-Pin_2): track 0.00 -> 42.9 mm
- net Net-(Driver1-PWMA): track 0.00 -> 39.9 mm, vias 0 -> 2
- net Net-(Driver2-PWMB): track 0.00 -> 38.1 mm, vias 0 -> 2
- net Net-(J5-Pin_1): track 0.00 -> 36.2 mm
- net Net-(Driver1-AI2): track 0.00 -> 34.3 mm, vias 0 -> 2
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- added copper zone on B.Cu, net GND
Other:
- board size 80 x 165 mm -> 80 x 166 mm
- board text added: "BF_1"
- board text added: "BF_2"
- board text added: "BF_P"
- board text added: "BL_1"
- board text added: "BL_2"
- board text added: "BL_P"
- board text added: "BR_1"
- board text added: "BR_2"
- board text added: "BR_P"
- board text added: "FR_1"
- board text added: "FR_2"
- board text added: "FR_P"
- board text added: "MCU GND"
- board text added: "MCU VCC"
- board text added: "PowerLatch"
- board text added: "SCL (ina219)"
- board text added: "SDA (ina219)"
- board text added: "STANDBY"
- board text added: "VCC"

Commit message: updated capacitor size
Parts:
- C1, C2, C3, C4, C6, C7: footprint Capacitor_SMD:C_0603_1608Metric_Pad1.08x0.95mm_HandSolder -> Capacitor_SMD:C_1206_3216Metric_Pad1.33x1.80mm_HandSolder
- moved C7 1.02 mm to (80.5, 87.1)
- moved C6 0.94 mm to (61.0, 86.9)
- moved C1 0.75 mm to (96.4, 91.0)
- moved C2 0.75 mm to (102.6, 91.0)
- moved C3 0.50 mm to (45.5, 91.5)
- renumbered 1A to OPM1, 1A to OPM2
Routing:
- net GND: track 2.53 -> 4.62 mm
- net Net-(Driver2-B01): track 30.7 -> 31.4 mm
