File: project/project.kicad_pcb (KiCad board)
At the start: 2 copper layers, 80 x 166 mm, 28 parts, among them J1 Conn_01x03, J2 Conn_02x07_Odd_Even, J3 Conn_01x02, J5 12V, Q1 IRF4905, Q2 NPN, SW1 SW_Push, U1 module_ina219

Commit message: added holes for mounting on the pcb
title
Routing:
- net /PowLatch: track 168.3 -> 158.4 mm, vias 2 -> 4
- net Net-(J3-Pin_1): track 147.2 -> 149.2 mm
Other:
- outline, holes or cut-outs redrawn
Changed lines of the file:
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@@
+	)
+	(gr_circle
+		(center 41.07 35.6)
+		(end 39.57 35.6)
+		(stroke
+			(width 0.2)
+			(type default)
+		)
+		(fill no)
+		(layer "Edge.Cuts")
+	)
+	(gr_circle
+		(center 41.07 163.1)
+		(end 41.1 161.6)
+		(stroke
+			(width 0.05)
+			(type default)
+		)
+		(fill no)
+		(layer "Edge.Cuts")
 	)
 	(gr_circle
 		(center 71.08575 108.6)
 		(end 71.08575 93.5)
+		(stroke
+			(width 0.05)
+			(type default)
+		)
+		(fill no)
+		(layer "Edge.Cuts")
+	)
+	(gr_circle
+		(center 101.1 35.599801)
+		(end 101.1 37.1)
+		(stroke
+			(width 0.05)
+			(type default)
+		)
+		(fill no)
+		(layer "Edge.Cuts")
+	)
+	(gr_circle
+		(center 101.1 163.1)
+		(end 102.6 163.1)
 		(stroke
 			(width 0.05)
@@
 	)
 	(segment
+		(start 33 69)
+		(end 51 51)
+		(width 1)
+		(layer "F.Cu")
+		(net "/PowLatch")
+	)
+	(segment
 		(start 46 127)
 		(end 46 145.5)
@@
 	)
 	(segment
-		(start 33 45)
-		(end 33 114)
+		(start 54 44)
+		(end 54 41.04)
+		(width 1)
+		(layer "F.Cu")
+		(net "/PowLatch")
+	)
+	(segment
+		(start 54 41.04)
+		(end 57.5 37.54)
 		(width 1)
 		(layer "F.Cu")
@@
 	)
 	(segment
-		(start 40.5 37.5)
-		(end 33 45)
-		(width 1)
-		(layer "F.Cu")
-		(net "/PowLatch")
-	)
-	(segment
-		(start 57.46 37.5)
-		(end 40.5 37.5)
-		(width 1)
-		(layer "F.Cu")
-		(net "/PowLatch")
-	)
-	(segment
 		(start 46 145.5)
 		(end 59.5 159)
@@
 		(net "/PowLatch")
 	)
+	(segment
+		(start 33 114)
+		(end 33 69)
+		(width 1)
+		(layer "F.Cu")
+		(net "/PowLatch")
+	)
 	(via
 		(at 59.5 159)
@@
 		(at 62.5 162)
 		(size 0.5)
+		(drill 0.3)
+		(layers "F.Cu" "B.Cu")
+		(net "/PowLatch")
+	)
+	(via
+		(at 54 44)
+		(size 0.6)
+		(drill 0.3)
+		(layers "F.Cu" "B.Cu")
+		(net "/PowLatch")
+	)
+	(via
+		(at 51 51)
+		(size 0.6)
 		(drill 0.3)
 		(layers "F.Cu" "B.Cu")
@@
 	)
 	(segment
+		(start 51 47)
+		(end 54 44)
+		(width 1)
+		(layer "B.Cu")
+		(net "/PowLatch")
+	)
+	(segment
+		(start 51 51)
+		(end 51 47)
+		(width 1)
+		(layer "B.Cu")
+		(net "/PowLatch")
+	)
+	(segment
 		(start 57.5 35)
 		(end 68.5 35)
@@
 	)
 	(segment
-		(start 98.5 36.5)
-		(end 107 45)
+		(start 107 45)
+		(end 103.7 41.7)
+		(width 0.4)
+		(layer "F.Cu")
+		(net "Net-(J3-Pin_2)")
+	)
+	(segment
+		(start 103.7 41.7)
+		(end 89.7 41.7)
 		(width 0.4)
 		(layer "F.Cu")
@@
 	)
 	(segment
-		(start 84.5 36.5)
-		(end 98.5 36.5)
-		(width 0.4)
-		(layer "F.Cu")
-		(net "Net-(J3-Pin_2)")
-	)
-	(segment
 		(start 77 146)
 		(end 75.88 146)
@@
 	)
 	(segment
+		(start 89.7 41.7)
+		(end 84.5 36.5)
+		(width 0.4)
+		(layer "F.Cu")
+		(net "Net-(J3-Pin_2)")
+	)
+	(segment
 		(start 75.88 146)
 		(end 75.745 145.865)
@@
 	)
 	(segment
+		(start 94.1 40.9)
+		(end 87.16 33.96)
+		(width 0.4)
+		(layer "F.Cu")
+		(net "Net-(J3-Pin_1)")
+	)
+	(segment
+		(start 104.4 40.9)
+		(end 94.1 40.9)
+		(width 0.4)
+		(layer "F.Cu")
+		(net "Net-(J3-Pin_1)")
+	)
+	(segment
 		(start 87.5 31.5)
 		(end 85.04 33.96)
@@
 	)
 	(segment
-		(start 95 31.5)
-		(end 87.5 31.5)
+		(start 87.16 33.96)
+		(end 84.5 33.96)
 		(width 0.4)
 		(layer "F.Cu")
@@
 	(segment
 		(start 108 44.5)
-		(end 95 31.5)
+		(end 104.4 40.9)
 		(width 0.4)
 		(layer "F.Cu")
@@
 		(polygon
 			(pts
-				(xy 31.5 28.5) (xy 111 28.5) (xy 111 188.5) (xy 31.5 188)
+				(xy 32.5 27.4) (xy 110.5 27.2) (xy 110.3 189.7) (xy 32.3 189.5) (xy 32.3 170.6)
 			)
 		)
