File: project/project.kicad_sch (KiCad schematic)
At the start: 0 parts

Commit message: v1
Parts:
- added J1, J2, J3, J4: Conn_01x02_Pin, Connector_JST:JST_XH_B2B-XH-A_1x02_P2.50mm_Vertical, symbol Connector:Conn_01x02_Pin
- added J5: Conn_01x02_Pin, SparkFun-Connectors:DEANS, symbol Connector:Conn_01x02_Pin
- added U1, U2: ROB-14450, ROB-14450:MODULE_ROB-14450, symbol ROB-14450:ROB-14450
Connections:
- new net: J3.1 (Pin_1), U2.4 (A01)
- new net: J3.2 (Pin_2), U2.5 (A02)
- new net: J1.1 (Pin_1), U1.4 (A01)
- new net: J1.2 (Pin_2), U1.5 (A02)
- new net: J2.2 (Pin_2), U1.6 (B02)
- new net: J2.1 (Pin_1), U1.7 (B01)
- new net: J4.2 (Pin_2), U2.6 (B02)
- new net: J4.1 (Pin_1), U2.7 (B01)
- new net +12V: J5.1 (Pin_1)
- new net GND: J5.2 (Pin_2), U1.3 (GND), U1.8 (GND), U1.9 (GND), U2.3 (GND), U2.8 (GND), U2.9 (GND)

Commit message: update
Parts:
- added C1, C2, C3, C4, C6, C7: 100nF, Capacitor_SMD:C_0603_1608Metric_Pad1.08x0.95mm_HandSolder, symbol Device:C_Small
- added C5: 100uF, Capacitor_THT:CP_Radial_D6.3mm_P2.50mm, symbol Device:C_Polarized_Small
- added J1: Conn_01x02_Pin, Connector_PinHeader_2.54mm:PinHeader_1x02_P2.54mm_Vertical, symbol Connector:Conn_01x02_Pin
- added J2: Conn_02x07_Odd_Even, Connector_PinHeader_2.54mm:PinHeader_2x07_P2.54mm_Vertical, symbol Connector_Generic:Conn_02x07_Odd_Even
- added J3: Conn_01x02, Connector_PinHeader_2.54mm:PinHeader_1x02_P2.54mm_Vertical, symbol Connector_Generic:Conn_01x02
- added StepDown_5V1: XL4015_Module, MC00100:XL4015_StepDown_Module, symbol MC00100:MC00100
- added StepDown_6V1: LM2596_Module, MC00100:CONV_MC00100, symbol MC00100:MC00100
- added U1: module_ina219, usini_sensors:module_ina219, symbol usini_sensors:module_ina219
- J5: value Conn_01x02_Pin -> 12V
- renumbered U2 to Driver1, U1 to Driver2, J1 to Motor1, J2 to Motor2, J3 to Motor3, J4 to Motor4
Connections:
- net GND: now also J5.- (Pin_2), C5.2, C6.1, C7.2, J1.1 (Pin_1), StepDown_5V1.IN-, StepDown_5V1.OUT-, StepDown_6V1.IN-, StepDown_6V1.OUT-, U1.2 (GND); no longer J5.2 (Pin_2)
- net at Driver1.4 (A01), Motor3.1 (Pin_1): now also C3.1
- net at Driver1.5 (A02), Motor3.2 (Pin_2): now also C3.2
- net VM: now reaches Driver2.1 (VM)
- net VM: now also Driver1.1 (VM), C5.1, StepDown_6V1.OUT+
- net at Driver2.10 (PWMB): now also J2.3 (Pin_3)
- net at Driver2.11 (BI2): now also J2.11 (Pin_11)
- net at Driver2.12 (BI1): now also J2.9 (Pin_9)
- net STANDBY: now reaches Driver2.13 (STBY)
- net STANDBY: now also Driver1.13 (STBY), J2.14 (Pin_14)
- net at Driver2.14 (AI1): now also J2.5 (Pin_5)
- net at Driver2.15 (AI2): now also J2.7 (Pin_7)
- net at Driver2.16 (PWMA): now also J2.1 (Pin_1)
- net VCC: now reaches Driver2.2 (VCC)
- net VCC: now also Driver1.2 (VCC), C6.2, C7.1, J2.13 (Pin_13), U1.1 (VCC)
- net at Driver2.4 (A01), Motor1.1 (Pin_1): now also C1.1
- net at Driver2.5 (A02), Motor1.2 (Pin_2): now also C1.2
- net at Driver2.6 (B02), Motor2.2 (Pin_2): now also C2.2
- net at Driver2.7 (B01), Motor2.1 (Pin_1): now also C2.1
- net at Driver1.10 (PWMB): now also J2.4 (Pin_4)
- net at Driver1.11 (BI2): now also J2.12 (Pin_12)
- net at Driver1.12 (BI1): now also J2.10 (Pin_10)
- net at Driver1.14 (AI1): now also J2.6 (Pin_6)
- net at Driver1.15 (AI2): now also J2.8 (Pin_8)
- net at Driver1.16 (PWMA): now also J2.2 (Pin_2)
- net at Driver1.6 (B02), Motor4.2 (Pin_2): now also C4.2
- net at Driver1.7 (B01), Motor4.1 (Pin_1): now also C4.1
- removed net +12V: J5.1 (Pin_1)
- new net: StepDown_5V1.IN+, StepDown_6V1.IN+, U1.5 (VIN-)
- new net: StepDown_6V1.MH1 (MOUTING), StepDown_6V1.MH2 (MOUTING)
- new net: J3.2 (Pin_2), U1.3 (SCL)
- new net: J3.1 (Pin_1), U1.4 (SDA)
- new net: J5.+ (Pin_1), U1.6 (VIN+)
- new net: StepDown_5V1.MH1 (MOUTING), StepDown_5V1.MH2 (MOUTING)
- new net: J1.2 (Pin_2), StepDown_5V1.OUT+
- no-connect marks 0 -> 2
Other:
- moved on the sheet: Driver1, Driver2, J5, Motor1, Motor2, Motor3, Motor4

Commit message: added latch
Parts:
- removed J1: Conn_01x02_Pin, Connector_PinHeader_2.54mm:PinHeader_1x02_P2.54mm_Vertical, symbol Connector:Conn_01x02_Pin
- added J1: Conn_01x03, Connector_PinHeader_2.54mm:PinHeader_1x03_P2.54mm_Vertical, symbol Connector_Generic:Conn_01x03
- added Q1: IRF4905, Package_TO_SOT_THT:TO-220-3_Vertical, symbol Transistor_FET:IRF4905
- added Q2: NPN, Package_TO_SOT_THT:TO-92_HandSolder, symbol Simulation_SPICE:NPN
- added R1, R2: 10k, Resistor_THT:R_Axial_DIN0309_L9.0mm_D3.2mm_P12.70mm_Horizontal, symbol Device:R
- added R3: 4.7k, Resistor_THT:R_Axial_DIN0309_L9.0mm_D3.2mm_P12.70mm_Horizontal, symbol Device:R
- added SW1: SW_Push, Button_Switch_THT:SW_PUSH-12mm, symbol Switch:SW_Push
Connections:
- net GND: now also J1.3 (Pin_3), Q2.3 (E), R2.1, SW1.1
- net at J5.+ (Pin_1): now also Q1.2 (D), R1.2; no longer U1.6 (VIN+)
- net at StepDown_5V1.OUT+: now also J1.2 (Pin_2)
- new net: Q1.1 (G), Q2.1 (C), R1.1, SW1.2
- new net: Q2.2 (B), R2.2, R3.2
- new net: Q1.3 (S), U1.6 (VIN+)
- new net PowLatch: J1.1 (Pin_1), R3.1
Other:
- moved on the sheet: C1, C2, C3, C4, C5, C6, C7, Driver1, Driver2, J2, J3, J5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

Commit message: last-update
Parts:
- added OPM1, OPM2: 1A, byRadu:OPM_Kuoyuh_91, symbol Switch:SW_SPST
Connections:
- net VM: now also OPM1.2 (B), OPM2.2 (B); no longer Driver1.1 (VM), Driver2.1 (VM)
- new net: Driver2.1 (VM), OPM1.1 (A)
- new net: Driver1.1 (VM), OPM2.1 (A)
Other:
- moved on the sheet: C5, J3, J5, Q1, Q2, R1, R2, R3, SW1, StepDown_5V1, StepDown_6V1, U1

Commit message: updated capacitor size
Parts:
- C1, C2, C3, C4, C6, C7: footprint Capacitor_SMD:C_0603_1608Metric_Pad1.08x0.95mm_HandSolder -> Capacitor_SMD:C_1206_3216Metric_Pad1.33x1.80mm_HandSolder
Changed lines of the file:
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@@
 			)
 		)
-		(property "Footprint" "Capacitor_SMD:C_0603_1608Metric_Pad1.08x0.95mm_HandSolder"
+		(property "Footprint" "Capacitor_SMD:C_1206_3216Metric_Pad1.33x1.80mm_HandSolder"
 			(at 189.23 250.19 0)
 			(hide yes)
@@
 			)
 		)
-		(property "Footprint" "Capacitor_SMD:C_0603_1608Metric_Pad1.08x0.95mm_HandSolder"
+		(property "Footprint" "Capacitor_SMD:C_1206_3216Metric_Pad1.33x1.80mm_HandSolder"
 			(at 213.36 250.19 0)
 			(hide yes)
@@
 			)
 		)
-		(property "Footprint" "Capacitor_SMD:C_0603_1608Metric_Pad1.08x0.95mm_HandSolder"
+		(property "Footprint" "Capacitor_SMD:C_1206_3216Metric_Pad1.33x1.80mm_HandSolder"
 			(at 166.37 250.19 0)
 			(hide yes)
@@
 			)
 		)
-		(property "Footprint" "Capacitor_SMD:C_0603_1608Metric_Pad1.08x0.95mm_HandSolder"
+		(property "Footprint" "Capacitor_SMD:C_1206_3216Metric_Pad1.33x1.80mm_HandSolder"
 			(at 138.43 168.91 0)
 			(hide yes)
@@
 			)
 		)
-		(property "Footprint" "Capacitor_SMD:C_0603_1608Metric_Pad1.08x0.95mm_HandSolder"
+		(property "Footprint" "Capacitor_SMD:C_1206_3216Metric_Pad1.33x1.80mm_HandSolder"
 			(at 137.16 210.82 0)
 			(hide yes)
@@
 			)
 		)
-		(property "Footprint" "Capacitor_SMD:C_0603_1608Metric_Pad1.08x0.95mm_HandSolder"
+		(property "Footprint" "Capacitor_SMD:C_1206_3216Metric_Pad1.33x1.80mm_HandSolder"
 			(at 143.51 250.19 0)
 			(hide yes)
